File: rOxpad-PCB/rOxpad.kicad_pcb (KiCad board)
At the start: 2 copper layers, 68.3 x 65.1 mm, 25 parts, among them SW1 SW_Push, U1 ATmega16U2-A, U2 PRTR5V0U2X, Y1 16MHz

Commit message: change MCU to atmega32u2
a lot cheaper
Parts:
- F1: value Polyfuse -> Polyfuse_Small
- R1, R2: value 22Ω -> 22
- R3, R4: value 10kΩ -> 10k
- R5, R6: value 5.1kΩ -> 5.1k
- U1: value ATmega16U2-A -> ATmega32U2-A
- USB1: footprint Type-C:HRO-TYPE-C-31-M-12-HandSoldering -> Connector_USB:USB_C_Receptacle_HRO_TYPE-C-31-M-12
Connections:
- C1 pad 1: Net-(C1-Pad1) -> unconnected-(C1-Pad1)
- R1 pad 2: Net-(R1-Pad2) -> unconnected-(R1-Pad2)
- R2 pad 2: Net-(R2-Pad2) -> unconnected-(R2-Pad2)
- U1 pad 1: XTAL1 -> unconnected-(U1-Pad1)
- U1 pad 19: KEY-0 -> unconnected-(U1-Pad19)
- U1 pad 2: XTAL2 -> unconnected-(U1-Pad2)
- U1 pad 20: KEY-1 -> unconnected-(U1-Pad20)
- U1 pad 21: KEY-2 -> unconnected-(U1-Pad21)
- U1 pad 24: Net-(R3-Pad2) -> unconnected-(U1-Pad24)
- U1 pad 27: Net-(C1-Pad1) -> unconnected-(U1-Pad27)
- U1 pad 29: Net-(R2-Pad2) -> unconnected-(U1-Pad29)
- U1 pad 3: GND -> unconnected-(U1-Pad3)
- U1 pad 30: Net-(R1-Pad2) -> unconnected-(U1-Pad30)
- U1 pad 32: +5V -> unconnected-(U1-Pad32)
- U1 pad 4: +5V -> unconnected-(U1-Pad4)
Routing:
- net unconnected-(U1-Pad29): track 0.00 -> 76.4 mm, vias 0 -> 2
- net Net-(R2-Pad2): track 76.4 -> 0.00 mm, vias 2 -> 0
- net unconnected-(R1-Pad2): track 0.00 -> 73.0 mm, vias 0 -> 2
- net Net-(R1-Pad2): track 73.0 -> 0.00 mm, vias 2 -> 0
- net unconnected-(C1-Pad1): track 0.00 -> 4.50 mm
- net Net-(C1-Pad1): track 4.50 -> 0.00 mm
